File: MidiController/PCB/MidiController.kicad_pcb (KiCad board)
At the start: 2 copper layers, 286.7 x 139.3 mm, 128 parts, among them J1 ST7735R, J2 AudioJack3, SW1 SW_Push_45deg, SW11 SW_Push_45deg, SW12 SW_Push_45deg, SW13 SW_Push_45deg, SW14 SW_Push_45deg, SW16 SW_Push_45deg, SW17 SW_Push_45deg, SW18 SW_Push_45deg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

Commit message: Update MidiController.kicad_pcb
Other:
- board text added: "FCK"
- board text added: "Made by Levi"
- board text added: "Midi-Keyboard"
- board text added: "NZS"
